File: PCB_IOT_SysIntel.kicad_sch (KiCad schematic)
At the start: 31 parts, among them J10 SSW-102-02-G-S, J11 SSW-102-02-G-S, J12 SSW-120-01-T-D, J13 SSW-102-02-G-S, J14 SSW-120-01-T-D, J15 SSW-102-02-G-S, J16 SSW-102-02-G-S, J17 SSW-102-02-G-S, J18 SSW-102-02-G-S, J19 SSW-102-02-G-S, J2 SSW-102-02-G-S, J20 SSW-102-02-G-S, J21 SSW-102-02-G-S, J22 SSW-102-02-G-S, J23 SSW-102-02-G-S, J24 SSW-102-02-G-S, J25 SSW-102-02-G-S, J26 SSW-120-01-T-D, J27 SSW-102-02-G-S, J28 SSW-102-02-G-S, J29 SSW-102-02-G-S, J3 SSW-102-02-G-S, J30 SSW-120-01-T-D, J4 SSW-102-02-G-S, J5 SSW-102-02-G-S, J6 SSW-102-02-G-S, J7 SSW-102-02-G-S, J8 SSW-102-02-G-S, J9 SSW-102-02-G-S, U1 RASPBERRY_PI_4B_4GB

Commit message: Project Version 1 Completed
Parts:
- removed J12, J14, J26, J30: SSW-120-01-T-D, SSW-120-01-T-D:SAMTEC_SSW-120-01-T-D, symbol 20PHeader:SSW-120-01-T-D
- added H1, H2, H3, H4: MountingHole, MountingHole:MountingHole_3.2mm_M3, symbol Mechanical:MountingHole
- added J15, J16, J29: SSW-125-01-T-D-LL, 25PHeader:SAMTEC_SSW-125-01-T-D-LL-Populated, symbol 25x2PHeader:SSW-125-01-T-D-LL
- added J30, J31, J32, J33, J34, J35, J36, J37, J38, J39, J40, J41, J42, J43, J44, J45, J46, J51, J52, J53, J54, J55, J56, J57, J58, J59, J60, J61, J62, J63, J64, J65: SSW-102-02-G-S, 1P_populated:SAMTEC_SSW-102-02-G-S-Populated, symbol 2PHeader:SSW-102-02-G-S
- added J47: SSW-125-01-T-D-LL, 25PHeader:SAMTEC_SSW-125-01-T-D-LL, symbol 25x2PHeader:SSW-125-01-T-D-LL
- added J48, J49, J50: SSW-130-01-T-D-LL, 30PHeader:SAMTEC_SSW-130-01-T-D-LL, symbol 30x2Pheader:SSW-130-01-T-D-LL
- J1: renamed from J22; footprint SSW-102-02-G-S:SAMTEC_SSW-102-02-G-S -> 1P_populated:SAMTEC_SSW-102-02-G-S-Populated
- J10: renamed from J23; footprint SSW-102-02-G-S:SAMTEC_SSW-102-02-G-S -> 1P_populated:SAMTEC_SSW-102-02-G-S-Populated
- J11: renamed from J27; footprint SSW-102-02-G-S:SAMTEC_SSW-102-02-G-S -> 1P_populated:SAMTEC_SSW-102-02-G-S-Populated
- J12: renamed from J28; footprint SSW-102-02-G-S:SAMTEC_SSW-102-02-G-S -> 1P_populated:SAMTEC_SSW-102-02-G-S-Populated
- J13: renamed from J29; footprint SSW-102-02-G-S:SAMTEC_SSW-102-02-G-S -> 1P_populated:SAMTEC_SSW-102-02-G-S-Populated
- J14: renamed from J1; footprint (none) -> M5Stack:M5Stack
- J17: renamed from J2; footprint SSW-102-02-G-S:SAMTEC_SSW-102-02-G-S -> 1P_populated:SAMTEC_SSW-102-02-G-S-Populated
- J18: renamed from J3; footprint SSW-102-02-G-S:SAMTEC_SSW-102-02-G-S -> 1P_populated:SAMTEC_SSW-102-02-G-S-Populated
- J19: renamed from J4; footprint SSW-102-02-G-S:SAMTEC_SSW-102-02-G-S -> 1P_populated:SAMTEC_SSW-102-02-G-S-Populated
- J2: renamed from J21; footprint SSW-102-02-G-S:SAMTEC_SSW-102-02-G-S -> 1P_populated:SAMTEC_SSW-102-02-G-S-Populated
- J20: renamed from J5; footprint SSW-102-02-G-S:SAMTEC_SSW-102-02-G-S -> 1P_populated:SAMTEC_SSW-102-02-G-S-Populated
- J21: renamed from J6; footprint SSW-102-02-G-S:SAMTEC_SSW-102-02-G-S -> 1P_populated:SAMTEC_SSW-102-02-G-S-Populated
- J22: renamed from J7; footprint SSW-102-02-G-S:SAMTEC_SSW-102-02-G-S -> 1P_populated:SAMTEC_SSW-102-02-G-S-Populated
- J23: renamed from J8; footprint SSW-102-02-G-S:SAMTEC_SSW-102-02-G-S -> 1P_populated:SAMTEC_SSW-102-02-G-S-Populated
- J24: renamed from J9; footprint SSW-102-02-G-S:SAMTEC_SSW-102-02-G-S -> 1P_populated:SAMTEC_SSW-102-02-G-S-Populated
- J25: renamed from J10; footprint SSW-102-02-G-S:SAMTEC_SSW-102-02-G-S -> 1P_populated:SAMTEC_SSW-102-02-G-S-Populated
- J26: renamed from J11; footprint SSW-102-02-G-S:SAMTEC_SSW-102-02-G-S -> 1P_populated:SAMTEC_SSW-102-02-G-S-Populated
- J27: renamed from J24; footprint SSW-102-02-G-S:SAMTEC_SSW-102-02-G-S -> 1P_populated:SAMTEC_SSW-102-02-G-S-Populated
- J28: renamed from J25; footprint SSW-102-02-G-S:SAMTEC_SSW-102-02-G-S -> 1P_populated:SAMTEC_SSW-102-02-G-S-Populated
- J3: renamed from J20; footprint SSW-102-02-G-S:SAMTEC_SSW-102-02-G-S -> 1P_populated:SAMTEC_SSW-102-02-G-S-Populated
- J4: renamed from J19; footprint SSW-102-02-G-S:SAMTEC_SSW-102-02-G-S -> 1P_populated:SAMTEC_SSW-102-02-G-S-Populated
- J5: renamed from J18; footprint SSW-102-02-G-S:SAMTEC_SSW-102-02-G-S -> 1P_populated:SAMTEC_SSW-102-02-G-S-Populated
- J6: renamed from J17; footprint SSW-102-02-G-S:SAMTEC_SSW-102-02-G-S -> 1P_populated:SAMTEC_SSW-102-02-G-S-Populated
- J7: renamed from J16; footprint SSW-102-02-G-S:SAMTEC_SSW-102-02-G-S -> 1P_populated:SAMTEC_SSW-102-02-G-S-Populated
- J8: renamed from J13; footprint SSW-102-02-G-S:SAMTEC_SSW-102-02-G-S -> 1P_populated:SAMTEC_SSW-102-02-G-S-Populated
- J9: renamed from J15; footprint SSW-102-02-G-S:SAMTEC_SSW-102-02-G-S -> 1P_populated:SAMTEC_SSW-102-02-G-S-Populated
- U1: footprint RASPBERRY_PI_4B_4GB:MODULE_RASPBERRY_PI_4B_4GB -> Raspberry:MODULE_RASPBERRY_PI_4B_4GB
Connections:
- net at J19.01, J19.02: now also J14.12 (Pin_12)
- net at J25.01, J25.02: now also J14.24 (Pin_24)
- net at J21.01, J21.02: now also J14.16 (Pin_16)
- net at J20.01, J20.02: now also J14.14 (Pin_14)
- net at J22.01, J22.02: now also J14.18 (Pin_18)
- net at J14.2 (Pin_2), J14.4 (Pin_4), J14.6 (Pin_6): now also J29.01, J29.02, J29.03, J29.04, J29.05, J29.06, J29.07, J29.08, J29.09, J29.10, J29.11, J29.12, J29.13, J29.14, J29.15, J29.16, J29.17, J29.18, J29.19, J29.20, J29.21, J29.22, J29.23, J29.24, J29.25, J29.26, J29.27, J29.28, J29.29, J29.30, J29.31, J29.32, J29.33, J29.34, J29.35, J29.36, J29.37, J29.38, J29.39, J29.40, J29.41, J29.42, J29.43, J29.44, J29.45, J29.46, J29.47, J29.48, J29.49, J29.50, J47.01, J47.02, J47.03, J47.04, J47.05, J47.06, J47.07, J47.08, J47.09, J47.10, J47.11, J47.12, J47.13, J47.14, J47.15, J47.16, J47.17, J47.18, J47.19, J47.20, J47.21, J47.22, J47.23, J47.24, J47.25, J47.26, J47.27, J47.28, J47.29, J47.30, J47.31, J47.32, J47.33, J47.34, J47.35, J47.36, J47.37, J47.38, J47.39, J47.40, J47.41, J47.42, J47.43, J47.44, J47.45, J47.46, J47.47, J47.48, J47.49, J47.50
- net at J23.01, J23.02: now also J14.20 (Pin_20)
- net at J17.01, J17.02: now also J14.8 (Pin_8)
- net at J14.11 (Pin_11): now also J15.01, J15.02, J15.03, J15.04, J15.05, J15.06, J15.07, J15.08, J15.09, J15.10, J15.11, J15.12, J15.13, J15.14, J15.15, J15.16, J15.17, J15.18, J15.19, J15.20, J15.21, J15.22, J15.23, J15.24, J15.25, J15.26, J15.27, J15.28, J15.29, J15.30, J15.31, J15.32, J15.33, J15.34, J15.35, J15.36, J15.37, J15.38, J15.39, J15.40, J15.41, J15.42, J15.43, J15.44, J15.45, J15.46, J15.47, J15.48, J15.49, J15.50
- net at J14.27 (Pin_27): now also J16.01, J16.02, J16.03, J16.04, J16.05, J16.06, J16.07, J16.08, J16.09, J16.10, J16.11, J16.12, J16.13, J16.14, J16.15, J16.16, J16.17, J16.18, J16.19, J16.20, J16.21, J16.22, J16.23, J16.24, J16.25, J16.26, J16.27, J16.28, J16.29, J16.30, J16.31, J16.32, J16.33, J16.34, J16.35, J16.36, J16.37, J16.38, J16.39, J16.40, J16.41, J16.42, J16.43, J16.44, J16.45, J16.46, J16.47, J16.48, J16.49, J16.50
- net at U1.1 (3V3), U1.17 (3V3): now also J50.01, J50.02, J50.03, J50.04, J50.05, J50.06, J50.07, J50.08, J50.09, J50.10, J50.11, J50.12, J50.13, J50.14, J50.15, J50.16, J50.17, J50.18, J50.19, J50.20, J50.21, J50.22, J50.23, J50.24, J50.25, J50.26, J50.27, J50.28, J50.29, J50.30, J50.31, J50.32, J50.33, J50.34, J50.35, J50.36, J50.37, J50.38, J50.39, J50.40, J50.41, J50.42, J50.43, J50.44, J50.45, J50.46, J50.47, J50.48, J50.49, J50.50, J50.51, J50.52, J50.53, J50.54, J50.55, J50.56, J50.57, J50.58, J50.59, J50.60
- net at U1.10 (GPIO15/RXD0): now also J52.01, J52.02
- net at U1.11 (GPIO17/GPIO_GEN0): now also J33.01, J33.02
- net at U1.12 (GPIO18/GPIO_GEN1): now also J35.01, J35.02
- net at U1.13 (GPIO27/GPIO_GEN2): now also J34.01, J34.02
- net at U1.14 (GND), U1.20 (GND), U1.25 (GND)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: now also J48.01, J48.02, J48.03, J48.04, J48.05, J48.06, J48.07, J48.08, J48.09, J48.10, J48.11, J48.12, J48.13, J48.14, J48.15, J48.16, J48.17, J48.18, J48.19, J48.20, J48.21, J48.22, J48.23, J48.24, J48.25, J48.26, J48.27, J48.28, J48.29, J48.30, J48.31, J48.32, J48.33, J48.34, J48.35, J48.36, J48.37, J48.38, J48.39, J48.40, J48.41, J48.42, J48.43, J48.44, J48.45, J48.46, J48.47, J48.48, J48.49, J48.50, J48.51, J48.52, J48.53, J48.54, J48.55, J48.56, J48.57, J48.58, J48.59, J48.60
- net at U1.15 (GPIO22/GPIO_GEN3): now also J36.01, J36.02
- net at U1.16 (GPIO23/GPIO_GEN4): now also J37.01, J37.02
- net at U1.18 (GPIO24/GPIO_GEN5): now also J38.01, J38.02
- net at U1.19 (GPIO10/SPI_MOSI): now also J43.01, J43.02
- net at U1.2 (5V), U1.4 (5V): now also J49.01, J49.02, J49.03, J49.04, J49.05, J49.06, J49.07, J49.08, J49.09, J49.10, J49.11, J49.12, J49.13, J49.14, J49.15, J49.16, J49.17, J49.18, J49.19, J49.20, J49.21, J49.22, J49.23, J49.24, J49.25, J49.26, J49.27, J49.28, J49.29, J49.30, J49.31, J49.32, J49.33, J49.34, J49.35, J49.36, J49.37, J49.38, J49.39, J49.40, J49.41, J49.42, J49.43, J49.44, J49.45, J49.46, J49.47, J49.48, J49.49, J49.50, J49.51, J49.52, J49.53, J49.54, J49.55, J49.56, J49.57, J49.58, J49.59, J49.60
- net at U1.21 (GPIO9/SPI_MISO): now also J44.01, J44.02
- net at U1.22 (GPIO25/GPIO_GEN6): now also J39.01, J39.02
- net at U1.23 (GPIO11/SPI_SCLK): now also J42.01, J42.02
- net at U1.24 (GPIO8/~{SPI_CE0}): now also J40.01, J40.02
- net at U1.26 (GPIO7/~{SPI_CE1}): now also J41.01, J41.02
- net at U1.27 (ID_SD): now also J45.01, J45.02
- net at U1.28 (ID_SC): now also J46.01, J46.02
- net at U1.29 (GPIO5): now also J53.01, J53.02
- net at U1.3 (GPIO2/SDA1): now also J30.01, J30.02
- net at U1.31 (GPIO6): now also J54.01, J54.02
- net at U1.32 (GPIO12): now also J55.01, J55.02
- net at U1.33 (GPIO13): now also J56.01, J56.02
- net at U1.35 (GPIO19): now also J58.01, J58.02
- net at U1.36 (GPIO16): now also J57.01, J57.02
- net at U1.37 (GPIO26): now also J61.01, J61.02
- net at U1.38 (GPIO20): now also J59.01, J59.02
- net at U1.40 (GPIO21): now also J60.01, J60.02
- net at U1.41 (TR01): now also J63.01, J63.02
- net at U1.42 (TR00): now also J62.01, J62.02
- net at U1.43 (TR03): now also J65.01, J65.02
- net at U1.44 (TR02): now also J64.01, J64.02
- net at U1.5 (GPIO3/SCL1): now also J31.01, J31.02
- net at U1.7 (GPIO4/GPIO_GCKL): now also J32.01, J32.02
- net at U1.8 (GPIO14/TXD0): now also J51.01, J51.02
- net at J24.01, J24.02: now also J14.22 (Pin_22)
- net at J26.01, J26.02: now also J14.26 (Pin_26)
- net at J28.01, J28.02: now also J14.30 (Pin_30)
- net at J27.01, J27.02: now also J14.28 (Pin_28)
- net at J14.10 (Pin_10): now also J18.01, J18.02
- no-connect marks 0 -> 1
Other:
- moved on the sheet: J17, J18, J19, J20, J21, J22, J23, J24, J25, J26, J27, J28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
